File: hardware/motor_side.brd (EAGLE design)
At the start: 16.5 x 47 mm, 11 parts, among them U1 MAX14870, U2 MAX14870

Commit message: Logo and name on tPlace/bPlace
Routing:
- net VIN: track 79.8 -> 83.7 mm
Other:
- board text added: "GND"
- board text added: "M_DIR"
- board text added: "M_PWM"
- board text added: "Motor"
- board text added: "S_DIR"
- board text added: "S_PWM"
- board text added: "Steering"
- board text added: "V1 2020 Motor Side"
- board text added: "VIN"
- board text removed: "Leonardo V1 (Motor side) Created by Isak Åslund Spring 2019"
- board text removed: "Leonardo V1 Motor Side"
